Commit message: add joint limits to position control

File: ultron/urdf/ultron.urdf (robot description, URDF)
Before this commit: robot ultron, 8 links, 7 joints
Joints:
- joint fixed: origin (none) -> xyz=0 0 0.0 rpy=0 0 0
- joint joint4: limit lower=-1.3 upper=1.3 effort=15.0 velocity=10. -> lower=-1.5 upper=1.5 effort=15.0 velocity=10.
- joint joint5: limit lower=-1.3 upper=1.3 effort=15.0 velocity=10.0 -> lower=-1.5 upper=1.5 effort=15.0 velocity=10.0

Commit message: add zero pos forward kinematics

File: ultron/urdf/ultron.urdf (robot description, URDF)
Before this commit: robot ultron, 8 links, 7 joints
Links:
- link link6: geometry visual mesh filename=package://ultron/meshes/link6.STL

Commit message: modify error to pos error and orientation error; se3 error is wrong cause Jacobian is not using se3 representation

File: ultron/urdf/ultron.urdf (robot description, URDF)
Before this commit: robot ultron, 8 links, 7 joints
Links:
- link link6: geometry collision box size=0.001 0.001 0.001; visual mesh filename=package://ultron/meshes/link6.STL

Commit message: change: change robot urdf to new arx 3

File: ultron/urdf/ultron.urdf (robot description, URDF)
Before this commit: robot ultron, 8 links, 7 joints
Links:
- link base_link: mass 0.44061 -> 0.44038
- link link1: mass 0.078442 -> 0.060835
- link link2: mass 1.073 -> 1.0733
- link link3: mass 0.50518 -> 0.4994
- link link4: mass 0.34332 -> 0.080971
- link link5: mass 0.33126 -> 0.60236
- link link6: mass 0.022383 -> 0.019531; geometry collision mesh filename=package://ultron/meshes/link6.STL; visual mesh filename=package://ultron/meshes/link6.STL
Joints:
- joint fixed: origin xyz=0 0 0.0 rpy=0 0 0 -> (none)
- joint joint2: origin xyz=0 0 0.0402 rpy=0 0 0 -> xyz=0.02 0 0.0402 rpy=0 0 0
- joint joint5: origin xyz=0.06 -0.002 0.0005 rpy=0 0 0 -> xyz=0.06575 -0.001 -0.0825 rpy=0 0 0
- joint joint6: origin xyz=0.078 0 -0.0005 rpy=3.1416 0 0 -> xyz=0.02845 0 0.0825 rpy=-3.1416 0 0
