Commit message: rename package to ultron_test

File: ultron_test/urdf/ultron.urdf (robot description, URDF)
Before this commit: robot ultron, 8 links, 7 joints
Links:
- link base_link: geometry collision mesh filename=package://ultron_test/meshes/base_link.STL; visual mesh filename=package://ultron_test/meshes/base_link.STL
- link link1: geometry collision mesh filename=package://ultron_test/meshes/link1.STL; visual mesh filename=package://ultron_test/meshes/link1.STL
- link link2: geometry collision mesh filename=package://ultron_test/meshes/link2.STL; visual mesh filename=package://ultron_test/meshes/link2.STL
- link link3: geometry collision mesh filename=package://ultron_test/meshes/link3.STL; visual mesh filename=package://ultron_test/meshes/link3.STL
- link link4: geometry collision mesh filename=package://ultron_test/meshes/link4.STL; visual mesh filename=package://ultron_test/meshes/link4.STL
- link link5: geometry collision mesh filename=package://ultron_test/meshes/link5.STL; visual mesh filename=package://ultron_test/meshes/link5.STL
- link link6: geometry collision mesh filename=package://ultron_test/meshes/link6.STL; visual mesh filename=package://ultron_test/meshes/link6.STL
