Commit message: add: current position to initial position movement

File: ultron_pos/urdf/ultron.urdf (robot description, URDF)
Before this commit: robot ultron, 8 links, 7 joints
Joints:
- joint joint4: limit lower=-1.5 upper=1.5 effort=15.0 velocity=10. -> lower=-1.57 upper=1.57 effort=15.0 velocity=10.
- joint joint5: limit lower=-1.5 upper=1.5 effort=15.0 velocity=10.0 -> lower=-1.57 upper=1.57 effort=15.0 velocity=10.0
